File: KalyPCB/KalyPCB.kicad_pcb (KiCad board)
At the start: 2 copper layers, 135.6 x 99.8 mm, 26 parts, among them J1 TRRS

Commit message: deconstruct
Parts:
- removed ?: , clipboard:1eb54394-d1bf-44fc-bfc9-1714e0e999b7
- removed J1: TRRS, Keebio-Parts:TRRS-PJ-320A
- removed S1, S2, S3: , PG1350
- added G*** (x3): LOGO, LOGO, F.Cu at (32.7, 185.2)
- added K1: KEYSW, Library:Kailh_socket_PG1350, F.Cu at (121.5, 140.9)
- added K10: KEYSW, Library:Kailh_socket_PG1350, F.Cu at (139.7, 191.4)
- added K11: KEYSW, Library:Kailh_socket_PG1350, F.Cu at (139.7, 208.3)
- added K12: KEYSW, Library:Kailh_socket_PG1350, F.Cu at (139.7, 225.1)
- added K13: KEYSW, Library:Kailh_socket_PG1350, F.Cu at (157.8, 140.9)
- added K14: KEYSW, Library:Kailh_socket_PG1350, F.Cu at (157.8, 157.7)
- added K15: KEYSW, Library:Kailh_socket_PG1350, F.Cu at (157.8, 174.6)
- added K16: KEYSW, Library:Kailh_socket_PG1350, F.Cu at (157.8, 191.4)
- added K17: KEYSW, Library:Kailh_socket_PG1350, F.Cu at (157.8, 208.3)
- added K18: KEYSW, Library:Kailh_socket_PG1350, F.Cu at (157.8, 225.1)
- added K19: KEYSW, Library:Kailh_socket_PG1350, F.Cu at (176.0, 140.9)
- added K2: KEYSW, Library:Kailh_socket_PG1350, F.Cu at (121.5, 157.7)
- added K20: KEYSW, Library:Kailh_socket_PG1350, F.Cu at (176.0, 157.7)
- added K21: KEYSW, Library:Kailh_socket_PG1350, F.Cu at (176.0, 174.6)
- added K22: KEYSW, Library:Kailh_socket_PG1350, F.Cu at (176.0, 191.4)
- added K23: KEYSW, Library:Kailh_socket_PG1350, F.Cu at (176.0, 208.3)
- added K24: KEYSW, Library:Kailh_socket_PG1350, F.Cu at (176.0, 225.1)
- added K25: KEYSW, Library:Kailh_socket_PG1350, F.Cu at (194.1, 140.9)
- added K26: KEYSW, Library:Kailh_socket_PG1350, F.Cu at (194.1, 157.7)
- added K27: KEYSW, Library:Kailh_socket_PG1350, F.Cu at (194.1, 174.6)
- added K28: KEYSW, Library:Kailh_socket_PG1350, F.Cu at (194.1, 191.4)
- added K29: KEYSW, Library:Kailh_socket_PG1350, F.Cu at (194.1, 208.3)
- added K3: KEYSW, Library:Kailh_socket_PG1350, F.Cu at (121.5, 174.6)
- added K30: KEYSW, Library:Kailh_socket_PG1350, F.Cu at (194.1, 225.1)
- added K31: KEYSW, Library:Kailh_socket_PG1350, F.Cu at (212.3, 140.9)
- added K32: KEYSW, Library:Kailh_socket_PG1350, F.Cu at (212.3, 157.7)
- added K33: KEYSW, Library:Kailh_socket_PG1350, F.Cu at (212.3, 174.6)
- added K34: KEYSW, Library:Kailh_socket_PG1350, F.Cu at (212.3, 191.4)
- added K35: KEYSW, Library:Kailh_socket_PG1350, F.Cu at (212.3, 208.3)
- added K36: KEYSW, Library:Kailh_socket_PG1350, F.Cu at (212.3, 225.1)
- added K4: KEYSW, Library:Kailh_socket_PG1350, F.Cu at (121.5, 191.4)
- added K5: KEYSW, Library:Kailh_socket_PG1350, F.Cu at (121.5, 208.3)
- added K6: KEYSW, Library:Kailh_socket_PG1350, F.Cu at (121.5, 225.1)
- added K7: KEYSW, Library:Kailh_socket_PG1350, F.Cu at (139.7, 140.9)
- added K8: KEYSW, Library:Kailh_socket_PG1350, F.Cu at (139.7, 157.7)
- added K9: KEYSW, Library:Kailh_socket_PG1350, F.Cu at (139.7, 174.6)
- added U1: ~, Library:pro_micro_rp2040, F.Cu at (128.7, 55.5)
- added U2: ~, Library:pro_micro_rp2040, F.Cu at (258.2, 190.5)
- moved G*** 96.8 mm to (35.8, 163.4) (x3)
Routing:
- net matrix_outer_bottom: track 169.6 -> 55.5 mm
- net matrix_index_bottom: track 92.2 -> 20.6 mm
- net matrix_middle_bottom: track 113.2 -> 43.4 mm
- net matrix_outer_top: track 129.4 -> 60.8 mm
- net matrix_inner_bottom: track 76.0 -> 7.69 mm
- net matrix_ring_bottom: track 128.5 -> 60.4 mm
- net matrix_pinky_bottom: track 149.1 -> 84.6 mm
- net thumb_inny: track 70.4 -> 7.73 mm
- net matrix_outer_home: track 133.4 -> 80.7 mm
- net matrix_index_top: track 60.7 -> 8.77 mm
- net matrix_middle_top: track 78.9 -> 28.7 mm
- net thumb_reachy: track 53.8 -> 4.13 mm
- net TX: track 48.7 -> 0.00 mm
- net matrix_ring_top: track 93.2 -> 44.8 mm
- net matrix_pinky_top: track 114.5 -> 67.1 mm
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Other:
- outline, holes or cut-outs redrawn
- board text removed: "Kaly42 V1"
- board text removed: "https://github.com/Dwctor/Kaly"

Commit message: mech ready
Parts:
- removed S10, S11, S12, S13, S14, S15, S16, S17, S18, S19, S20, S21, S4, S5, S6, S7, S8, S9: , PG1350
- added MB1: MountingHole, Library:MountingHole_2.2mm_M2-8mm, F.Cu at (122.6, 162.3)
- added U3: TRRS, Keebio-Parts:TRRS-PJ-320A, F.Cu at (124.2, 20.8)
- added U4: TRRS, Keebio-Parts:TRRS-PJ-320A, F.Cu at (174.0, 20.8)
- moved K23 188.1 mm to (258.2, 39.1)
- moved K5 187.8 mm to (40.0, 39.1)
- moved K24 179.0 mm to (186.1, 46.4)
- moved K6 179.0 mm to (112.0, 46.4)
- moved K22 177.0 mm to (240.1, 26.4)
- moved K4 176.8 mm to (58.0, 26.4)
- moved U2 172.3 mm to (153.3, 53.8)
- moved K12 170.9 mm to (94.0, 60.5)
- moved K10 168.1 mm to (40.0, 56.1)
- moved K30 164.9 mm to (204.2, 60.5)
- moved K21 159.7 mm to (222.2, 21.7)
- moved K3 159.5 mm to (76.0, 21.7)
- moved K15 156.2 mm to (39.4, 72.7)
- moved K18 154.8 mm to (101.6, 80.9), turned to -15 degrees
- moved K9 154.5 mm to (58.0, 43.5)
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Connections:
- K1 pad 1: unconnected-(K1-Pad1) -> GND
- K1 pad 2: /K1 -> /L01
- K10 pad 1: unconnected-(K10-Pad1) -> GND
- K10 pad 2: unconnected-(K10-Pad2) -> /L10
- K11 pad 1: unconnected-(K11-Pad1) -> GND
- K11 pad 2: unconnected-(K11-Pad2) -> /L11
- K12 pad 1: unconnected-(K12-Pad1) -> GND
- K12 pad 2: unconnected-(K12-Pad2) -> /L12
- K13 pad 1: unconnected-(K13-Pad1) -> GND
- K13 pad 2: unconnected-(K13-Pad2) -> /L13
- K14 pad 1: unconnected-(K14-Pad1) -> GND
- K14 pad 2: unconnected-(K14-Pad2) -> /L14
- K15 pad 1: unconnected-(K15-Pad1) -> GND
- K15 pad 2: unconnected-(K15-Pad2) -> /L15
- K16 pad 1: unconnected-(K16-Pad1) -> GND
- K16 pad 2: unconnected-(K16-Pad2) -> /L16
- K17 pad 1: unconnected-(K17-Pad1) -> GND
- K17 pad 2: unconnected-(K17-Pad2) -> /L17
- K18 pad 1: unconnected-(K18-Pad1) -> GND
- K18 pad 2: unconnected-(K18-Pad2) -> /L18
- K19 pad 1: unconnected-(K19-Pad1) -> GND
- K19 pad 2: unconnected-(K19-Pad2) -> /R01
- K2 pad 1: unconnected-(K2-Pad1) -> GND
- K2 pad 2: unconnected-(K2-Pad2) -> /L02
- K20 pad 1: unconnected-(K20-Pad1) -> GND
- K20 pad 2: unconnected-(K20-Pad2) -> /R02
- K21 pad 1: unconnected-(K21-Pad1) -> GND
- K21 pad 2: unconnected-(K21-Pad2) -> /R03
- K22 pad 1: unconnected-(K22-Pad1) -> GND
- K22 pad 2: unconnected-(K22-Pad2) -> /R04
- K23 pad 1: unconnected-(K23-Pad1) -> GND
- K23 pad 2: unconnected-(K23-Pad2) -> /R05
- K24 pad 1: unconnected-(K24-Pad1) -> GND
- K24 pad 2: unconnected-(K24-Pad2) -> /R06
- K25 pad 1: unconnected-(K25-Pad1) -> GND
- K25 pad 2: unconnected-(K25-Pad2) -> /R07
- K26 pad 1: unconnected-(K26-Pad1) -> GND
- K26 pad 2: unconnected-(K26-Pad2) -> /R08
- K27 pad 1: unconnected-(K27-Pad1) -> GND
- K27 pad 2: unconnected-(K27-Pad2) -> /R09
- K28 pad 1: unconnected-(K28-Pad1) -> GND
- K28 pad 2: unconnected-(K28-Pad2) -> /R10
- K29 pad 1: unconnected-(K29-Pad1) -> GND
- K29 pad 2: unconnected-(K29-Pad2) -> /R11
- K3 pad 1: unconnected-(K3-Pad1) -> GND
- K3 pad 2: unconnected-(K3-Pad2) -> /L03
- K30 pad 1: unconnected-(K30-Pad1) -> GND
- K30 pad 2: unconnected-(K30-Pad2) -> /R12
- K31 pad 1: unconnected-(K31-Pad1) -> GND
- K31 pad 2: unconnected-(K31-Pad2) -> /R13
- K32 pad 1: unconnected-(K32-Pad1) -> GND
- K32 pad 2: unconnected-(K32-Pad2) -> /R14
- K33 pad 1: unconnected-(K33-Pad1) -> GND
- K33 pad 2: unconnected-(K33-Pad2) -> /R15
- K34 pad 1: unconnected-(K34-Pad1) -> GND
- K34 pad 2: unconnected-(K34-Pad2) -> /R16
- K35 pad 1: unconnected-(K35-Pad1) -> GND
- K35 pad 2: unconnected-(K35-Pad2) -> /R17
- K36 pad 1: unconnected-(K36-Pad1) -> GND
- K36 pad 2: unconnected-(K36-Pad2) -> /R18
- K4 pad 1: unconnected-(K4-Pad1) -> GND
- K4 pad 2: unconnected-(K4-Pad2) -> /L04
- K5 pad 1: unconnected-(K5-Pad1) -> GND
- K5 pad 2: unconnected-(K5-Pad2) -> /L05
- K6 pad 1: unconnected-(K6-Pad1) -> GND
- K6 pad 2: unconnected-(K6-Pad2) -> /L06
- K7 pad 1: unconnected-(K7-Pad1) -> GND
- K7 pad 2: unconnected-(K7-Pad2) -> /L07
- K8 pad 1: unconnected-(K8-Pad1) -> GND
- K8 pad 2: unconnected-(K8-Pad2) -> /L08
- K9 pad 1: unconnected-(K9-Pad1) -> GND
- K9 pad 2: unconnected-(K9-Pad2) -> /L09
- U2 pad 28: unconnected-(U2-GP28-Pad28) -> /R02
- U2 pad 29: unconnected-(U2-GP29-Pad29) -> /R01
Routing:
- net matrix_pinky_bottom: track 84.6 -> 0.00 mm
- net matrix_pinky_home: track 84.2 -> 0.00 mm
- net matrix_outer_home: track 80.7 -> 0.00 mm
- net matrix_ring_home: track 67.7 -> 0.00 mm
- net matrix_pinky_top: track 67.1 -> 0.00 mm
- net matrix_outer_top: track 60.8 -> 0.00 mm
- net matrix_ring_bottom: track 60.4 -> 0.00 mm
- net matrix_outer_bottom: track 55.5 -> 0.00 mm
- net matrix_middle_home: track 53.0 -> 0.00 mm
- net matrix_ring_top: track 44.8 -> 0.00 mm
- net matrix_middle_bottom: track 43.4 -> 0.00 mm
- net matrix_middle_top: track 28.7 -> 0.00 mm
- net matrix_index_home: track 26.4 -> 0.00 mm
- net matrix_index_bottom: track 20.6 -> 0.00 mm
- net matrix_inner_top: track 10.6 -> 0.00 mm
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Other:
- board size 135.6 x 99.8 mm -> 240.2 x 99.8 mm

Commit message: gitteg thert
Parts:
- added MB10: MountingHole, Library:MountingHole_2.2mm_M2-8mm, F.Cu at (237.6, 156.9)
- added MB2: MountingHole, Library:MountingHole_2.2mm_M2-8mm, F.Cu at (123.6, 38.0)
- added MB3: MountingHole, Library:MountingHole_2.2mm_M2-8mm, F.Cu at (48.8, 38.0)
- added MB4: MountingHole, Library:MountingHole_2.2mm_M2-8mm, F.Cu at (48.8, 75.0)
- added MB5: MountingHole, Library:MountingHole_2.2mm_M2-8mm, F.Cu at (96.5, 146.7)
- added MB6: MountingHole, Library:MountingHole_2.2mm_M2-8mm, F.Cu at (174.6, 75.0)
- added MB7: MountingHole, Library:MountingHole_2.2mm_M2-8mm, F.Cu at (174.6, 38.0)
- added MB8: MountingHole, Library:MountingHole_2.2mm_M2-8mm, F.Cu at (249.8, 38.0)
- added MB9: MountingHole, Library:MountingHole_2.2mm_M2-8mm, F.Cu at (249.8, 75.0)
- moved MB1 87.3 mm to (123.6, 75.0)
- turned K33 to 180 degrees
- turned K34 to -46 degrees
Connections:
- U1 pad 0: unconnected-(U1-GP0-Pad0) -> /LTX
- U1 pad 1: unconnected-(U1-GP1-Pad1) -> /LRX
- U1 pad 10: unconnected-(U1-GP10-Pad10) -> /L03
- U1 pad 2: /K1 -> /L01
- U1 pad 3: unconnected-(U1-GP3-Pad3) -> /L02
- U1 pad 4: unconnected-(U1-GP4-Pad4) -> /L04
- U1 pad 5: unconnected-(U1-GP5-Pad5) -> /L05
- U1 pad 5V: unconnected-(U1-Pad5V) -> /LVCC
- U1 pad 6: unconnected-(U1-GP6-Pad6) -> /L06
- U1 pad 7: unconnected-(U1-GP7-Pad7) -> /L07
- U1 pad 8: unconnected-(U1-GP8-Pad8) -> /L08
- U1 pad 9: unconnected-(U1-GP9-Pad9) -> /L09
- U2 pad 0: unconnected-(U2-GP0-Pad0) -> /RTX
- U2 pad 1: unconnected-(U2-GP1-Pad1) -> /RRX
- U2 pad 5V: unconnected-(U2-Pad5V) -> /RVCC
- U3 pad 1: unconnected-(U3-SLEEVE-Pad1) -> GND
- U3 pad 2: unconnected-(U3-TIP-Pad2) -> /LVCC
- U3 pad 3: unconnected-(U3-RING1-Pad3) -> /LTX
- U3 pad 4: unconnected-(U3-RING2-Pad4) -> /LRX
- U4 pad 1: unconnected-(U4-SLEEVE-Pad1) -> GND
- U4 pad 2: unconnected-(U4-TIP-Pad2) -> /RVCC
- U4 pad 3: unconnected-(U4-RING1-Pad3) -> /RRX
- U4 pad 4: unconnected-(U4-RING2-Pad4) -> /RTX
Routing:
- net /L09: track 0.00 -> 85.3 mm
- net /L04: track 0.00 -> 84.5 mm
- net /L03: track 0.00 -> 69.9 mm
- net /L08: track 0.00 -> 69.1 mm
- net /L05: track 0.00 -> 64.4 mm
- net /L02: track 0.00 -> 48.8 mm
- net /L07: track 0.00 -> 48.4 mm
- net /L01: track 0.00 -> 28.0 mm
- net /L06: track 0.00 -> 9.00 mm
- net GND: vias 0 -> 5
Other:
- board text removed: "By: Kael S.A."
- board text removed: "Kaly42"
