File: KalyPCB/KalyPCB.kicad_sch (KiCad schematic)
At the start: 38 parts, among them K1 KEYSW, K10 KEYSW, K11 KEYSW, K12 KEYSW, K13 KEYSW, K14 KEYSW, K15 KEYSW, K16 KEYSW, K17 KEYSW, K18 KEYSW, K19 KEYSW, K2 KEYSW, K20 KEYSW, K21 KEYSW, K22 KEYSW, K23 KEYSW, K24 KEYSW, K25 KEYSW, K26 KEYSW, K27 KEYSW, K28 KEYSW, K29 KEYSW, K3 KEYSW, K30 KEYSW, K31 KEYSW, K32 KEYSW, K33 KEYSW, K34 KEYSW, K35 KEYSW, K36 KEYSW, K4 KEYSW, K5 KEYSW, K6 KEYSW, K7 KEYSW, K8 KEYSW, K9 KEYSW

Commit message: mech ready
Parts:
- added MB1: MountingHole, Library:MountingHole_2.2mm_M2-8mm, symbol New_Library:MountingHole
- added U3, U4: TRRS, Keebio-Parts:TRRS-PJ-320A, symbol keebio:TRRS
- renumbered K22 to K20, K25 to K21, K29 to K22, K33 to K23, K20 to K24, K23 to K25, K30 to K27, K34 to K28, K21 to K29, K24 to K30, K27 to K31, K31 to K32, K35 to K33, K28 to K34, K32 to K35
Connections:
- net GND: now also K1.1, K10.1, K11.1, K12.1, K13.1, K14.1, K15.1, K16.1, K17.1, K18.1, K19.1, K2.1, K20.1, K21.1, K22.1, K23.1, K24.1, K25.1, K26.1, K27.1, K28.1, K29.1, K3.1, K30.1, K31.1, K32.1, K33.1, K34.1, K35.1, K36.1, K4.1, K5.1, K6.1, K7.1, K8.1, K9.1
- net K1: no longer K1.2
- net R10: now reaches K28.2
- net L03: now reaches K3.2
- net L15: now reaches K15.2
- net R02: now reaches U2.28 (GP28)
- net R02: now also K20.2
- net R01: now reaches U2.29 (GP29)
- net R01: now also K19.2
- net L02: now reaches K2.2
- net R06: now reaches K24.2
- net L14: now reaches K14.2
- net L11: now reaches K11.2
- net L07: now reaches K7.2
- net L18: now reaches K18.2
- net L06: now reaches K6.2
- net R08: now reaches K26.2
- net L13: now reaches K13.2
- net L16: now reaches K16.2
- net R05: now reaches K23.2
- net R14: now reaches K32.2
- net L08: now reaches K8.2
- net R16: now reaches K34.2
- net L05: now reaches K5.2
- net L04: now reaches K4.2
- net R12: now reaches K30.2
- net R11: now reaches K29.2
- net R18: now reaches K36.2
- net R03: now reaches K21.2
- net L09: now reaches K9.2
- net L12: now reaches K12.2
- net R07: now reaches K25.2
- net L10: now reaches K10.2
- net R17: now reaches K35.2
- net R13: now reaches K31.2
- net L17: now reaches K17.2
- net R09: now reaches K27.2
- net R04: now reaches K22.2
- net R15: now reaches K33.2
- new net L01: K1.2

Commit message: gitteg thert
Parts:
- added MB10, MB2, MB3, MB4, MB5, MB6, MB7, MB8, MB9: MountingHole, Library:MountingHole_2.2mm_M2-8mm, symbol New_Library:MountingHole
Connections:
- net K1 is gone; now on net L01: U1.2 (GP2)
- net GND: now also U3.1 (SLEEVE), U4.1 (SLEEVE)
- net L02: now also U1.3 (GP3)
- net L03: now also U1.10 (GP10)
- net L04: now also U1.4 (GP4)
- net L05: now also U1.5 (GP5)
- net L06: now also U1.6 (GP6)
- net L07: now also U1.7 (GP7)
- net L08: now also U1.8 (GP8)
- net L09: now also U1.9 (GP9)
- net RTX: now reaches U2.0 (GP0)
- net RTX: now also U4.4 (RING2)
- net RRX: now reaches U2.1 (GP1)
- net RRX: now also U4.3 (RING1)
- net RVCC: now reaches U2.5V
- net RVCC: now also U4.2 (TIP)
- net LTX: now reaches U1.0 (GP0)
- net LTX: now also U3.3 (RING1)
- net LRX: now reaches U1.1 (GP1)
- net LRX: now also U3.4 (RING2)
- net LVCC: now reaches U1.5V
- net LVCC: now also U3.2 (TIP)
